Commit message: feat: add lidar link and joint to G23 URDF, update save_images.sh

File: src/syncai_bringup/description/G23.urdf (robot description, URDF)
Before this commit: robot G23, 17 links, 16 joints
Links:
- added link laser, mass 0.01
Joints:
- added joint laser_joint: type fixed, parent base_link, child laser, origin xyz=0.195 0.00 0.155 rpy=0 0.25 0

Commit message: feat: update configuration and parameters for improved robot functionality

File: src/syncai_bringup/description/G23.urdf (robot description, URDF)
Before this commit: robot G23, 17 links, 16 joints
Links:
- added link lidar_top
Joints:
- added joint lidar_top_joint: type fixed, parent base_link, child lidar_top, origin xyz=0.195 0.00 0.155 rpy=0 0.25 0
