Commit message: feat(bringup): parent camera_optical_frame on lidar_top (provisional)
The camera's optical frame was a root in the global TF tree: G23.urdf had
no camera link, so no image could be transformed into base_link. A fixed
camera_optical_joint under lidar_top now carries robot01's camera pose,
measured by hand (7 cm ahead of and 6.5 cm below the lidar along the body
axes, level, facing forward) and expressed in the 0.25 rad-pitched
lidar_top as xyz 0.084 0 -0.046, rpy -1.3208 0 -1.5708.

It is provisional: a tape measure is good to a cm or two and a few
degrees, enough for TF lookups and an rviz check, not for projecting
lidar points onto the image. It hangs off lidar_top rather than
base_link because the lidar-camera calibration that replaces it solves
camera <-> lidar, and since the Livox driver now stamps raw clouds with
lidar_top, that result goes into the joint as it is.

camera_imu_link is still a root (publish_imu has to stay false). The
bringup launch comment and README said the URDF had no camera link and
were updated.

Co-Authored-By: Claude Opus 5.5 <noreply@anthropic.com>

File: src/syncai_bringup/description/G23.urdf (robot description, URDF)
Before this commit: robot G23, 18 links, 17 joints
Links:
- added link camera_optical_frame
Joints:
- added joint camera_optical_joint: type fixed, parent lidar_top, child camera_optical_frame, origin xyz=0.084 0.0 -0.046 rpy=-1.3208 0 -1.5708

Commit message: fix(bringup): split lidar_top into the lidar and its IMU, stamp clouds with it
lidar_top stood for two points ~5 cm apart: syncai_lio_bridge (and
syncai_robot_state) map the Point-LIO body pose through it as if it were the
body, while the raw cloud was stamped with a separate <robot_id>/laser that
nothing parented. Point-LIO's body frame is the MID360's built-in IMU, not
the lidar: it broadcasts r_wi / t_wi and moves every point into the IMU frame
through r_il / t_il. That is why 06721b7 (stamp clouds with lidar_top) was
reverted in f522212.

The URDF now has both: lidar_top is the lidar itself (the origin of its
points), and lidar_top_imu hangs under it at -t_il, the inverse of the
extrinsic in pointlio_params.yaml, which it has to mirror. With that, the
Livox driver stamps livox/lidar with <robot_id>/lidar_top, so a raw cloud
transforms into the robot tree, and a camera <-> lidar calibration result goes
into camera_optical_joint as it is. Point-LIO ignores the header, so LIO is
unaffected; bags recorded before this carry <robot_id>/laser.

Cross-repository: syncai_lio_bridge and syncai_robot_state still name
lidar_top as their lidar_frame, which is numerically what they looked up
before, so nothing changes until they move to lidar_top_imu in their own
repositories; that move removes the ~5 cm (~2.3 cm planar) offset.

Dead or misleading frame names cleaned up on the way:
- planner_server.launch.py: the scan source's sensor_frame was
  <robot_id>/laser, a frame nothing broadcast; it is <robot_id>/scan, as in
  controller_server's launch. No data reaches that source on the 3D stack.
- syncai_localizer: local_frame is now overridden with
  <robot_id>/pointlio_odom in the launch, and the YAML placeholder is
  pointlio_odom instead of laser. The 10 ms timer broadcasts map ->
  local_frame from startup, so until pointlio's first message an unprefixed
  map -> laser was on TF.
- syncai_pointlio: the YAML fallbacks are pointlio_odom / pointlio_body
  (the fork's lidar / body before), matching what pgo_node derives in a bare
  run; README and launch no longer claim the body frame is the lidar.
- bringup.yaml: drop a sentence about the camera params block removed in #42.

No code changes: the URDF, launch and params files are symlinked under
--symlink-install, so restarting the bringup and localization panes applies
it without a rebuild.

Co-Authored-By: Claude Opus 5.5 <noreply@anthropic.com>

File: src/syncai_bringup/description/G23.urdf (robot description, URDF)
Before this commit: robot G23, 19 links, 18 joints
Links:
- added link lidar_top_imu
Joints:
- added joint lidar_top_imu_joint: type fixed, parent lidar_top, child lidar_top_imu, origin xyz=0.011 0.02329 -0.04412 rpy=0 0 0

Commit message: fix(bringup): calibrated camera_optical_joint rotation for robot01
rpy -1.3208 0 -1.5708 -> -1.3240 -0.0060 -1.5868: a rotation-only NID fit
on two static bags (pos01 + pos02) with the new equidistant intrinsics,
mostly a 0.8 deg pan to the right that the tape measure could not see
(0.73 / 0.89 deg on each bag alone). Each bag's rotation cut the other
bag's horizontal edge residual from 9-11 px to ~4 px.

xyz stays the tape measure: on these scenes the 6-DoF fits moved the camera
4-27 cm in directions that disagreed, and mis-projected a robot lying 1.2 m
away by ~100 px. G23.urdf is shared by the fleet, so the joint is robot01's
until a per-robot override exists.

Co-Authored-By: Claude Opus 5.5 <noreply@anthropic.com>

File: src/syncai_bringup/description/G23.urdf (robot description, URDF)
Before this commit: robot G23, 20 links, 19 joints
Joints:
- joint camera_optical_joint: origin xyz=0.084 0.0 -0.046 rpy=-1.3208 0 -1.5708 -> xyz=0.084 0.0 -0.046 rpy=-1.3240 -0.0060 -1.5868
